Commit message: feat: add mujoco and rviz files.

File: urdf/magicdog_w.urdf (robot description, URDF)
Before this commit: robot magicdog, 18 links, 17 joints
Links:
- link FL_calf: geometry collision box size=0.28885 0.025 0.025; visual mesh filename=package://magicdog-w_description/meshes/magicdog_left_knee_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 scale=1 1 1
- link FL_hip: geometry collision cylinder length=0.07 radius=0.05; visual mesh filename=package://magicdog-w_description/meshes/magicdog_abad.stl scale=1 1 1
- link FL_thigh: geometry collision box size=0.1 0.03 0.04; visual mesh filename=package://magicdog-w_description/meshes/magicdog_hip.stl scale=1 1 1
- link FL_wheel: geometry collision cylinder length=0.030 radius=0.090; visual mesh filename=package://magicdog-w_description/meshes/magicdog_left_wheel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 scale=1 1 1
- link FR_calf: geometry collision box size=0.28885 0.025 0.025; visual mesh filename=package://magicdog-w_description/meshes/magicdog_right_knee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 scale=1 1 1
- link FR_hip: geometry collision cylinder length=0.07 radius=0.05; visual mesh filename=package://magicdog-w_description/meshes/magicdog_abad.stl scale=1 1 1
- link FR_thigh: geometry collision box size=0.1 0.03 0.04; visual mesh filename=package://magicdog-w_description/meshes/magicdog_hip_right.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 scale=1 1 1
- link FR_wheel: geometry collision cylinder length=0.030 radius=0.090; visual mesh filename=package://magicdog-w_description/meshes/magicdog_right_whee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 scale=1 1 1
- link RL_calf: geometry collision box size=0.28885 0.025 0.025; visual mesh filename=package://magicdog-w_description/meshes/magicdog_left_knee_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 scale=1 1 1
- link RL_hip: geometry collision cylinder length=0.07 radius=0.05; visual mesh filename=package://magicdog-w_description/meshes/magicdog_abad.stl scale=1 1 1
- link RL_thigh: geometry collision box size=0.1 0.03 0.04; visual mesh filename=package://magicdog-w_description/meshes/magicdog_hip.stl scale=1 1 1
- link RL_wheel: geometry collision cylinder length=0.030 radius=0.090; visual mesh filename=package://magicdog-w_description/meshes/magicdog_left_wheel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 scale=1 1 1
- link RR_calf: geometry collision box size=0.28885 0.025 0.025; visual mesh filename=package://magicdog-w_description/meshes/magicdog_right_knee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 scale=1 1 1
- link RR_hip: geometry collision cylinder length=0.07 radius=0.05; visual mesh filename=package://magicdog-w_description/meshes/magicdog_abad.stl scale=1 1 1
- link RR_thigh: geometry collision box size=0.1 0.03 0.04; visual mesh filename=package://magicdog-w_description/meshes/magicdog_hip_right.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 scale=1 1 1
- link RR_wheel: geometry collision cylinder length=0.030 radius=0.090; visual mesh filename=package://magicdog-w_description/meshes/magicdog_right_whee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 scale=1 1 1
- link base: geometry collision box size=0.327 0.194 0.114; visual mesh filename=package://magicdog-w_description/meshes/magicdog_base.stl scale=1 1 1
Joints:
- joint FL_wheel_joint: type revolute -> continuous
- joint FR_wheel_joint: type revolute -> continuous
- joint RL_wheel_joint: type revolute -> continuous
- joint RR_wheel_joint: type revolute -> continuous
